Commit message: Add middle finger virtual link to g1 models

File: assets/unitree_g1/g1_29dof_w_hands.urdf (robot description, URDF)
Before this commit: robot g1_23dof_lock_wrist, 39 links, 38 joints
Links:
- added link left_hand_middle_0_link
- added link right_hand_middle_0_link
Joints:
- added joint left_hand_middle_0_joint: type fixed, parent left_wrist_yaw_link, child left_hand_middle_0_link, origin xyz=0.1192 0.0046 -0.0285 rpy=0 0 0
- added joint right_hand_middle_0_joint: type fixed, parent right_wrist_yaw_link, child right_hand_middle_0_link, origin xyz=0.1192 -0.0046 -0.0285 rpy=0 0 0

Commit message: Bugfixes on motion projection

File: assets/unitree_g1/g1_29dof_w_hands.urdf (robot description, URDF)
Before this commit: robot g1_23dof_lock_wrist, 41 links, 40 joints
Joints:
- joint left_hand_middle_0_joint: origin xyz=0.1192 0.0046 -0.0285 rpy=0 0 0 -> xyz=0.1192 -0.0186 0.0285 rpy=0 0 0
- joint right_hand_middle_0_joint: origin xyz=0.1192 -0.0046 -0.0285 rpy=0 0 0 -> xyz=0.1192 0.0186 0.0285 rpy=0 0 0
